Commit message: added box bot sample

File: pechan_gazebo_sim/description/robot/box_bot.xacro (robot description, xacro)
@@ -15,8 +15,12 @@
   -->
   <xacro:box_bot_body parent_name="${base_name}"/>
-  <xacro:link_wheel name="right_wheel" r="${wheel_radius}" l="${wheel_width}" incr="${wheel_increment}"/>
+  <!-- <xacro:link_wheel name="right_wheel" r="${wheel_radius}" l="${wheel_width}" incr="${wheel_increment}"/>
   <xacro:joint_wheel name="joint_right_wheel" parent="${base_name}" child="right_wheel" origin_xyz="0 ${base_box_x / 2.0} ${-1.0 * wheel_radius}" />
   <xacro:link_wheel name="left_wheel" r="${wheel_radius}" l="${wheel_width}" incr="${wheel_increment}"/>
-  <xacro:joint_wheel name="joint_left_wheel" parent="${base_name}" child="left_wheel" origin_xyz="0 ${-1.0 * base_box_x / 2.0} ${-1.0 * wheel_radius}" />
+  <xacro:joint_wheel name="joint_left_wheel" parent="${base_name}" child="left_wheel" origin_xyz="0 ${-1.0 * base_box_x / 2.0} ${-1.0 * wheel_radius}" /> -->
+  <xacro:link_wheel name="right_wheel" r="${wheel_radius}" l="${wheel_width}" incr="${wheel_increment}"/>
+  <xacro:joint_wheel name="joint_right_wheel" parent="${base_name}" child="right_wheel" origin_xyz="0 ${-1.0 * base_box_x / 2.0} ${-1.0 * wheel_radius}" />
+  <xacro:link_wheel name="left_wheel" r="${wheel_radius}" l="${wheel_width}" incr="${wheel_increment}"/>
+  <xacro:joint_wheel name="joint_left_wheel" parent="${base_name}" child="left_wheel" origin_xyz="0 ${base_box_x / 2.0} ${-1.0 * wheel_radius}" />
   <xacro:caster_wheel parent="chassis" caster_wheel_name="front" origin_xyz="${(base_box_x / 2.0) - wheel_increment} 0 ${-1.0* base_box_x / 2.0}" radius="${wheel_increment}" length="${dummy_length}"/>
   <xacro:caster_wheel parent="chassis" caster_wheel_name="back" origin_xyz="${(-1.0 *base_box_x / 2.0) + wheel_increment} 0 ${-1.0* base_box_x / 2.0}" radius="${wheel_increment}" length="${dummy_length}"/>

File: pechan_gazebo_sim/description/robot/properties.xacro (robot description, xacro)
@@ -11,5 +11,6 @@
     <!-- Wheels -->
 	<xacro:property name="wheel_radius" value="${base_box_z / 4.0}"/>
-    <xacro:property name="wheel_width" value="0.001"/>
+    <!-- <xacro:property name="wheel_width" value="0.001"/> -->
+    <xacro:property name="wheel_width" value="0.005"/>
     <xacro:property name="wheel_increment" value="0.010"/>
     <xacro:property name="mu1_wheel" value="0.5"/>

File: pechan_gazebo_sim/description/robot/wheels.xacro (robot description, xacro)
@@ -2,5 +2,5 @@
 <robot xmlns:xacro="http://www.ros.org/wiki/xacro">
     <!-- Wheels-->
-    <xacro:macro  name="link_wheel" params="name r l incr">
+  <xacro:macro  name="link_wheel" params="name r l incr">
       <link name="${name}">
           <inertial>
